Commit message: preliminary changes to enable 2 gripper setup, will need to test on hardware

File: robotiq_description/urdf/robotiq_2f_85_gripper.urdf.xacro (robot description, xacro)
@@ -2,9 +2,22 @@
 <robot xmlns:xacro="http://wiki.ros.org/xacro" name="robotiq_gripper">
     <!-- parameters -->
-    <xacro:arg name="use_fake_hardware" default="true" />
+    <xacro:arg name="use_fake_hardware" default="true"/>
+    <xacro:arg name="com_port_robot_1" default="/dev/ttyACM0" />
+    <xacro:arg name="com_port_robot_2" default="/dev/ttyACM1" />
     <!-- Import macros -->
     <xacro:include filename="$(find robotiq_description)/urdf/robotiq_2f_85_macro.urdf.xacro" />
     <link name="world" />
-    <xacro:robotiq_gripper name="RobotiqGripperHardwareInterface" prefix="" parent="world" use_fake_hardware="$(arg use_fake_hardware)">
+    <xacro:robotiq_gripper name="RobotiqGripperHardwareInterface"
+                            prefix="robot1/"
+                            parent="world"
+                            use_fake_hardware="$(arg use_fake_hardware)"
+                            com_port="$(arg com_port_robot_1)">
+        <origin xyz="2.0 0 0" rpy="0 0 0" />
+    </xacro:robotiq_gripper>
+    <xacro:robotiq_gripper name="RobotiqGripperHardwareInterface"
+                          prefix="robot2/"
+                          parent="world"
+                          use_fake_hardware="$(arg use_fake_hardware)"
+                          com_port="$(arg com_port_robot_2)">
         <origin xyz="0 0 0" rpy="0 0 0" />
     </xacro:robotiq_gripper>
